File: switch-control-hat/switch-control-hat.kicad_pcb (KiCad board)
At the start: 2 copper layers, 85 x 56 mm, 39 parts, among them J1 Conn_01x13, J2 Conn_01x03, J3 Conn_01x02, P1 Conn_02x20_Odd_Even, U1 TLP3543, U2 TLP3543, U3 TLP3543, U4 TLP3543, U5 TLP3543, U6 TLP3543, U7 TLP3543, U8 TLP3543, U9 DS3231M

Commit message: Add files via upload
Updated PCB
Parts:
- moved J3 2.54 mm to (278.7, 138.6)
Routing:
- net GND: track 2.02 -> 380.9 mm, vias 0 -> 9
- net /GPIO2(SDA1): track 6.90 -> 104.2 mm
- net +3V3: track 17.9 -> 93.3 mm
- net /GPIO3(SCL1): track 3.75 -> 76.7 mm
- net Net-(BT1-Pad1): track 9.35 -> 28.3 mm
- net +12V: track 201.1 -> 192.8 mm
- net +5V: track 0.00 -> 2.54 mm
- net Net-(J3-Pad2): track 19.6 -> 17.0 mm
- net Net-(J3-Pad1): track 17.7 -> 15.2 mm
- net /POS1: track 48.2 -> 50.1 mm
- net /POS3: track 49.0 -> 50.2 mm
- net /POS5: track 48.1 -> 48.8 mm

Commit message: Further updated PCB
Parts:
- added REF**: TerminalBlock_bornier-3_P5.08mm, TerminalBlock:TerminalBlock_bornier-3_P5.08mm, F.Cu at (269.9, 161.4)
- added REF**: TerminalBlock_bornier-5_P5.08mm, TerminalBlock:TerminalBlock_bornier-5_P5.08mm, F.Cu at (240.6, 161.4)
- added REF**: TerminalBlock_bornier-6_P5.08mm, TerminalBlock:TerminalBlock_bornier-6_P5.08mm, F.Cu at (210.2, 161.4)
- moved D3 0.76 mm to (220.3, 134.8)
Routing:
- net GND: track 380.9 -> 395.7 mm, vias 9 -> 5
- net /POS5: track 48.8 -> 62.3 mm
- net /RESET: track 47.6 -> 51.4 mm
- net /POS6: track 29.3 -> 31.1 mm
- net /GPIO2(SDA1): track 104.2 -> 105.2 mm
- net /NOISE-DIODE: track 30.4 -> 31.2 mm
