File: switch-control-hat/switch-control-hat.sch (KiCad schematic (older format))
At the start: 39 parts, among them J1 Conn_01x13, J2 Conn_01x03, J3 Conn_01x02, P1 Conn_02x20_Odd_Even, U1 TLP3543, U2 TLP3543, U3 TLP3543, U4 TLP3543, U5 TLP3543, U6 TLP3543, U7 TLP3543, U8 TLP3543, U9 DS3231M

Commit message: Final board layout
Parts:
- J1: footprint Connector_Phoenix_MC:PhoenixContact_MC_1,5_13-G-3.5_1x13_P3.50mm_Horizontal -> Connector_Phoenix_MC:PhoenixContact_MC_1,5_13-G-3.81_1x13_P3.81mm_Horizontal
- J2: footprint Connector_Phoenix_MC:PhoenixContact_MC_1,5_3-G-3.5_1x03_P3.50mm_Horizontal -> Connector_Phoenix_MC:PhoenixContact_MC_1,5_3-G-3.81_1x03_P3.81mm_Horizontal
Connections:
- net labels added: GNDA, GPIO18(GEN1)(PWM0)
- net labels removed: GPIO4(GCLK)
- wire segments 196 -> 197
- no-connect marks 13 -> 12
Changed lines of the file:
@@
 Text Label 750  1200 0    50   ~ 0
 GPIO3(SCL1)
-Text Label 750  1300 0    50   ~ 0
-GPIO4(GCLK)
 Text Label 750  1500 0    50   ~ 0
 GPIO17(GEN0)
@@
 	1    0    0    -1
 $EndComp
-$Comp
-L Connector_Generic:Conn_02x20_Odd_Even P1
-U 1 1 59AD464A
-P 2100 1900
-F 0 "P1" H 2150 3017 50  0000 C CNN
-F 1 "Conn_02x20_Odd_Even" H 2150 2926 50  0000 C CNN
-F 2 "Connector_PinSocket_2.54mm:PinSocket_2x20_P2.54mm_Vertical" H -2750 950 50  0001 C CNN
-F 3 "" H -2750 950 50  0001 C CNN
-	1    2100 1900
-	1    0    0    -1
-$EndComp
 Wire Wire Line
 	2400 2900 3450 2900
@@
 Wire Wire Line
 	8900 1600 9200 1600
-Text Label 8900 1800 2    50   ~ 0
+Text Label 8900 1200 2    50   ~ 0
 ONE-WIRE
 Wire Wire Line
-	8900 1800 9200 1800
-$Comp
-L power:GND #PWR0117
-U 1 1 5D2B92E3
-P 9050 2350
-F 0 "#PWR0117" H 9050 2100 50  0001 C CNN
-F 1 "GND" H 9055 2177 50  0000 C CNN
-F 2 "" H 9050 2350 50  0001 C CNN
-F 3 "" H 9050 2350 50  0001 C CNN
-	1    9050 2350
-	1    0    0    -1
-$EndComp
+	8900 1200 9200 1200
 $Comp
 L Device:D_ALT D8
@@
 	0    -1   -1   0
 $EndComp
-$Comp
-L power:GND #PWR0118
-U 1 1 5D14880F
-P 9950 6150
-F 0 "#PWR0118" H 9950 5900 50  0001 C CNN
-F 1 "GND" H 9955 5977 50  0000 C CNN
-F 2 "" H 9950 6150 50  0001 C CNN
-F 3 "" H 9950 6150 50  0001 C CNN
-	1    9950 6150
-	1    0    0    -1
-$EndComp
 Wire Wire Line
 	9950 6000 9950 6150
@@
 	0    -1   -1   0
 $EndComp
-$Comp
-L power:GND #PWR0119
-U 1 1 5D1A4C97
-P 6650 5400
-F 0 "#PWR0119" H 6650 5150 50  0001 C CNN
-F 1 "GND" H 6655 5227 50  0000 C CNN
-F 2 "" H 6650 5400 50  0001 C CNN
-F 3 "" H 6650 5400 50  0001 C CNN
-	1    6650 5400
-	1    0    0    -1
-$EndComp
 Wire Wire Line
 	6650 5250 6650 5400
@@
 	0    -1   -1   0
 $EndComp
-$Comp
-L power:GND #PWR0120
-U 1 1 5D2296A7
-P 9950 4850
-F 0 "#PWR0120" H 9950 4600 50  0001 C CNN
-F 1 "GND" H 9955 4677 50  0000 C CNN
-F 2 "" H 9950 4850 50  0001 C CNN
-F 3 "" H 9950 4850 50  0001 C CNN
-	1    9950 4850
-	1    0    0    -1
-$EndComp
 Wire Wire Line
 	9950 4700 9950 4850
@@
 	0    -1   -1   0
 $EndComp
-$Comp
-L power:GND #PWR0121
-U 1 1 5D264A56
-P 6650 4150
-F 0 "#PWR0121" H 6650 3900 50  0001 C CNN
-F 1 "GND" H 6655 3977 50  0000 C CNN
-F 2 "" H 6650 4150 50  0001 C CNN
-F 3 "" H 6650 4150 50  0001 C CNN
-	1    6650 4150
-	1    0    0    -1
-$EndComp
 Wire Wire Line
 	6650 4000 6650 4150
@@
 	0    -1   -1   0
 $EndComp
-$Comp
-L power:GND #PWR0122
-U 1 1 5D2CE3D8
-P 9950 3600
-F 0 "#PWR0122" H 9950 3350 50  0001 C CNN
-F 1 "GND" H 9955 3427 50  0000 C CNN
-F 2 "" H 9950 3600 50  0001 C CNN
-F 3 "" H 9950 3600 50  0001 C CNN
-	1    9950 3600
-	1    0    0    -1
-$EndComp
 Wire Wire Line
 	9950 3450 9950 3600
@@
 	0    -1   -1   0
 $EndComp
-$Comp
-L power:GND #PWR0123
-U 1 1 5D335BFD
-P 6650 2850
-F 0 "#PWR0123" H 6650 2600 50  0001 C CNN
-F 1 "GND" H 6655 2677 50  0000 C CNN
-F 2 "" H 6650 2850 50  0001 C CNN
-F 3 "" H 6650 2850 50  0001 C CNN
-	1    6650 2850
-	1    0    0    -1
-$EndComp
 Wire Wire Line
 	6650 2700 6650 2850
@@
 	0    -1   -1   0
 $EndComp
-$Comp
-L power:GND #PWR0124
-U 1 1 5D3A7212
-P 6650 6650
-F 0 "#PWR0124" H 6650 6400 50  0001 C CNN
-F 1 "GND" H 6655 6477 50  0000 C CNN
-F 2 "" H 6650 6650 50  0001 C CNN
-F 3 "" H 6650 6650 50  0001 C CNN
-	1    6650 6650
-	1    0    0    -1
-$EndComp
 Wire Wire Line
 	6650 6500 6650 6650
@@
 	0    -1   -1   0
 $EndComp
-$Comp
-L power:GND #PWR0125
-U 1 1 5D3AFCAE
-P 6650 1600
-F 0 "#PWR0125" H 6650 1350 50  0001 C CNN
-F 1 "GND" H 6655 1427 50  0000 C CNN
-F 2 "" H 6650 1600 50  0001 C CNN
-F 3 "" H 6650 1600 50  0001 C CNN
-	1    6650 1600
-	1    0    0    -1
-$EndComp
 Wire Wire Line
 	6650 1450 6650 1600
@@
 F 0 "J1" H 9480 1642 50  0000 L CNN
 F 1 "Conn_01x13" H 9480 1551 50  0000 L CNN
-F 2 "Connector_Phoenix_MC:PhoenixContact_MC_1,5_13-G-3.5_1x13_P3.50mm_Horizontal" H 9400 1600 50  0001 C CNN
+F 2 "Connector_Phoenix_MC:PhoenixContact_MC_1,5_13-G-3.81_1x13_P3.81mm_Horizontal" H 9400 1600 50  0001 C CNN
 F 3 "~" H 9400 1600 50  0001 C CNN
 	1    9400 1600
 	1    0    0    -1
 $EndComp
-NoConn ~ 2400 2100
-NoConn ~ 1900 2100
-NoConn ~ 1900 2000
-NoConn ~ 1900 1900
-NoConn ~ 1900 2300
-NoConn ~ 2400 2300
-NoConn ~ 2400 1500
-NoConn ~ 2400 1700
-NoConn ~ 1900 1700
-NoConn ~ 1900 1600
-NoConn ~ 2400 1800
-NoConn ~ 2400 2200
-NoConn ~ 2400 2000
 $Comp
 L Connector_Generic:Conn_01x03 J2
@@
 F 0 "J2" H 2518 6775 50  0000 C CNN
 F 1 "Conn_01x03" H 2518 6866 50  0000 C CNN
-F 2 "Connector_Phoenix_MC:PhoenixContact_MC_1,5_3-G-3.5_1x03_P3.50mm_Horizontal" H 2600 7100 50  0001 C CNN
+F 2 "Connector_Phoenix_MC:PhoenixContact_MC_1,5_3-G-3.81_1x03_P3.81mm_Horizontal" H 2600 7100 50  0001 C CNN
 F 3 "~" H 2600 7100 50  0001 C CNN
 	1    2600 7100
 	-1   0    0    1
-$EndComp
-$Comp
-L power:GND #PWR0126
-U 1 1 5DE7FC83
-P 2950 7000
-F 0 "#PWR0126" H 2950 6750 50  0001 C CNN
-F 1 "GND" V 2955 6872 50  0000 R CNN
-F 2 "" H 2950 7000 50  0001 C CNN
-F 3 "" H 2950 7000 50  0001 C CNN
-	1    2950 7000
-	0    -1   -1   0
 $EndComp
 $Comp
@@
 	9050 2350 9050 2000
 Wire Wire Line
-	9050 1200 9200 1200
-Wire Wire Line
 	9200 2000 9050 2000
 Connection ~ 9050 2000
 Wire Wire Line
-	9050 1200 9050 1400
-Wire Wire Line
 	9050 1400 9200 1400
-Connection ~ 9050 1400
-Wire Wire Line
-	9050 1400 9050 2000
-Text Label 4850 1000 2    50   ~ 0
-GPIO5
+Wire Wire Line
+	9050 1400 9050 1800
 Wire Wire Line
 	4850 1000 5000 1000
-Text Label 4850 3550 2    50   ~ 0
-GPIO6
 Wire Wire Line
 	4850 2250 5000 2250
@@
 Text Label 8150 3000 2    50   ~ 0
 GPIO19(SPI1_MISO)
+Text Label 8150 5550 2    50   ~ 0
+GPIO26
+Wire Wire Line
+	4850 4800 5000 4800
+Wire Wire Line
+	4850 6050 5000 6050
 Text Label 8150 4250 2    50   ~ 0
-GPIO26
-Wire Wire Line
-	4850 4800 5000 4800
-Wire Wire Line
-	4850 6050 5000 6050
-Text Label 8150 5550 2    50   ~ 0
 GPIO20(SPI1_MOSI)
 Text Label 4850 6050 2    50   ~ 0
 GPIO16
+Wire Wire Line
+	8150 5550 8300 5550
+Wire Wire Line
+	8300 4250 8150 4250
+Wire Wire Line
+	8150 3000 8300 3000
+$Comp
+L power:GNDA #PWR0117
+U 1 1 5D2250E5
+P 2950 7000
+F 0 "#PWR0117" H 2950 6750 50  0001 C CNN
+F 1 "GNDA" V 2955 6872 50  0000 R CNN
+F 2 "" H 2950 7000 50  0001 C CNN
+F 3 "" H 2950 7000 50  0001 C CNN
+	1    2950 7000
+	0    -1   -1   0
+$EndComp
+$Comp
+L power:GNDA #PWR0118
+U 1 1 5D238D3E
+P 9050 2350
+F 0 "#PWR0118" H 9050 2100 50  0001 C CNN
+F 1 "GNDA" H 9055 2177 50  0000 C CNN
+F 2 "" H 9050 2350 50  0001 C CNN
+F 3 "" H 9050 2350 50  0001 C CNN
+	1    9050 2350
+	1    0    0    -1
+$EndComp
+$Comp
+L power:GNDA #PWR0119
+U 1 1 5D245700
+P 9950 3600
+F 0 "#PWR0119" H 9950 3350 50  0001 C CNN
+F 1 "GNDA" H 9955 3427 50  0000 C CNN
+F 2 "" H 9950 3600 50  0001 C CNN
+F 3 "" H 9950 3600 50  0001 C CNN
+	1    9950 3600
+	1    0    0    -1
+$EndComp
+$Comp
+L power:GNDA #PWR0120
+U 1 1 5D25123E
+P 9950 4850
+F 0 "#PWR0120" H 9950 4600 50  0001 C CNN
+F 1 "GNDA" H 9955 4677 50  0000 C CNN
+F 2 "" H 9950 4850 50  0001 C CNN
+F 3 "" H 9950 4850 50  0001 C CNN
+	1    9950 4850
+	1    0    0    -1
+$EndComp
+$Comp
+L power:GNDA #PWR0121
+U 1 1 5D25C237
+P 9950 6150
+F 0 "#PWR0121" H 9950 5900 50  0001 C CNN
+F 1 "GNDA" H 9955 5977 50  0000 C CNN
+F 2 "" H 9950 6150 50  0001 C CNN
+F 3 "" H 9950 6150 50  0001 C CNN
+	1    9950 6150
+	1    0    0    -1
+$EndComp
+$Comp
+L power:GNDA #PWR0122
+U 1 1 5D2671CF
+P 6650 5400
+F 0 "#PWR0122" H 6650 5150 50  0001 C CNN
+F 1 "GNDA" H 6655 5227 50  0000 C CNN
+F 2 "" H 6650 5400 50  0001 C CNN
+F 3 "" H 6650 5400 50  0001 C CNN
+	1    6650 5400
+	1    0    0    -1
+$EndComp
+$Comp
+L power:GNDA #PWR0123
+U 1 1 5D2767E4
+P 6650 6650
+F 0 "#PWR0123" H 6650 6400 50  0001 C CNN
+F 1 "GNDA" H 6655 6477 50  0000 C CNN
+F 2 "" H 6650 6650 50  0001 C CNN
+F 3 "" H 6650 6650 50  0001 C CNN
+	1    6650 6650
+	1    0    0    -1
+$EndComp
+$Comp
+L power:GNDA #PWR0124
+U 1 1 5D282F37
+P 6650 4150
+F 0 "#PWR0124" H 6650 3900 50  0001 C CNN
+F 1 "GNDA" H 6655 3977 50  0000 C CNN
+F 2 "" H 6650 4150 50  0001 C CNN
+F 3 "" H 6650 4150 50  0001 C CNN
+	1    6650 4150
+	1    0    0    -1
+$EndComp
+$Comp
+L power:GNDA #PWR0125
+U 1 1 5D29294B
+P 6650 2850
+F 0 "#PWR0125" H 6650 2600 50  0001 C CNN
+F 1 "GNDA" H 6655 2677 50  0000 C CNN
+F 2 "" H 6650 2850 50  0001 C CNN
+F 3 "" H 6650 2850 50  0001 C CNN
+	1    6650 2850
+	1    0    0    -1
+$EndComp
+$Comp
+L power:GNDA #PWR0126
+U 1 1 5D29E75B
+P 6650 1600
+F 0 "#PWR0126" H 6650 1350 50  0001 C CNN
+F 1 "GNDA" H 6655 1427 50  0000 C CNN
+F 2 "" H 6650 1600 50  0001 C CNN
+F 3 "" H 6650 1600 50  0001 C CNN
+	1    6650 1600
+	1    0    0    -1
+$EndComp
+$Comp
+L Connector_Generic:Conn_02x20_Odd_Even P1
+U 1 1 59AD464A
+P 2100 1900
+F 0 "P1" H 2150 3017 50  0000 C CNN
+F 1 "Conn_02x20_Odd_Even" H 2150 2926 50  0000 C CNN
+F 2 "Connector_PinSocket_2.54mm:PinSocket_2x20_P2.54mm_Vertical" H -2750 950 50  0001 C CNN
+F 3 "" H -2750 950 50  0001 C CNN
+	1    2100 1900
+	1    0    0    -1
+$EndComp
+NoConn ~ 1900 1900
+NoConn ~ 1900 2000
+NoConn ~ 2400 2100
+NoConn ~ 1900 2100
+NoConn ~ 1900 1600
+NoConn ~ 1900 1700
+NoConn ~ 2400 1700
+NoConn ~ 2400 1800
+NoConn ~ 2400 2000
+NoConn ~ 2400 2200
+NoConn ~ 2400 2300
+NoConn ~ 1900 2300
+Text Label 750  1300 0    50   ~ 0
+ONE-WIRE
+Text Label 3450 1500 2    50   ~ 0
+GPIO18(GEN1)(PWM0)
+Wire Wire Line
+	2400 1500 3450 1500
+Text Label 4850 1000 2    50   ~ 0
+GPIO18(GEN1)(PWM0)
 Text Label 4850 2250 2    50   ~ 0
+GPIO17(GEN0)
+Text Label 4850 3550 2    50   ~ 0
 GPIO12(PWM0)
 Wire Wire Line
-	8150 5550 8300 5550
-Wire Wire Line
-	8300 4250 8150 4250
-Wire Wire Line
-	8150 3000 8300 3000
+	9200 1800 9050 1800
+Connection ~ 9050 1800
+Wire Wire Line
+	9050 1800 9050 2000
 $EndSCHEMATC

Commit message: Fixed error where optoisolators output was connected in reverse
Connections:
- wire segments 197 -> 189
Other:
- moved on the sheet: D1, D2, D3, D4, D5, D6, D7, D8

Commit message: Added pullup resistor for one-wire interface and changed 13 pin connector to 12 pin
Parts:
- removed J1: Conn_01x13, Connector_Phoenix_MC:PhoenixContact_MC_1,5_13-G-3.81_1x13_P3.81mm_Horizontal, symbol Connector_Generic:Conn_01x13
- added J1: Frontend Connector, Connector_Phoenix_MC:PhoenixContact_MC_1,5_12-G-3.81_1x12_P3.81mm_Horizontal, symbol Connector_Generic:Conn_01x12
- added R13: 4K7, Resistor_SMD:R_0603_1608Metric_Pad1.05x0.95mm_HandSolder, symbol Device:R_US
- BT1: value Battery_Cell -> 3V
- C1: value C -> 1uF; footprint Capacitor_SMD:C_0805_2012Metric -> Capacitor_SMD:C_0603_1608Metric_Pad1.05x0.95mm_HandSolder
- D1, D2, D3, D4, D5, D6, D7, D8: value D_ALT -> 1N4001
- J2: value Conn_01x03 -> Power Connector
- P1: value Conn_02x20_Odd_Even -> RPi-Header
- R1, R2, R3, R4, R5, R6, R7, R8: value R_US -> 200; footprint Resistor_SMD:R_0805_2012Metric -> Resistor_SMD:R_0603_1608Metric_Pad1.05x0.95mm_HandSolder
- R10, R11, R12, R9: value R_US -> 4K7; footprint Resistor_SMD:R_0805_2012Metric -> Resistor_SMD:R_0603_1608Metric_Pad1.05x0.95mm_HandSolder
Connections:
- wire segments 189 -> 188

Commit message: Final verision of schematic and PCB layout
Connections:
- net GND: now also D1.1 (K), D2.1 (K), D3.1 (K), D4.1 (K), D5.1 (K), D6.1 (K), D7.1 (K), D8.1 (K), J1.10 (Pin_10)
- net GNDA: no longer D1.1 (K), D2.1 (K), D3.1 (K), D4.1 (K), D5.1 (K), D6.1 (K), D7.1 (K), D8.1 (K), J1.10 (Pin_10)
- net GPIO12(PWM0): now also R2.2; no longer R3.2
- net GPIO13(PWM1): now also R3.2; no longer R4.2
- net GPIO16: now also R4.2; no longer R5.2
- net GPIO19(SPI1_MISO): now also R5.2; no longer R6.2
- net GPIO20(SPI1_MOSI): now also R6.2; no longer R7.2
- net GPIO21(SPI1_SCK): now also R8.2
- net GPIO26: now also R7.2; no longer R8.2
- net GPIO6: now also R1.2
- net GPIO17(GEN0): no longer names the net of P1.11 (Pin_11)
- net GPIO17(GEN0): no longer R2.2
- net GPIO18(GEN1)(PWM0): no longer names the net of P1.12 (Pin_12)
- net GPIO18(GEN1)(PWM0): no longer R1.2
- no-connect marks 12 -> 14
Changed lines of the file:
@@
 EESchema Schematic File Version 4
 LIBS:switch-control-hat-cache
-EELAYER 29 0
+EELAYER 30 0
 EELAYER END
 $Descr A4 11693 8268
@@
 Wire Wire Line
 	4850 2250 5000 2250
-Text Label 4850 4800 2    50   ~ 0
+Text Label 4850 3550 2    50   ~ 0
 GPIO13(PWM1)
 Wire Wire Line
 	4850 3550 5000 3550
-Text Label 8150 3000 2    50   ~ 0
+Text Label 4850 6050 2    50   ~ 0
 GPIO19(SPI1_MISO)
-Text Label 8150 5550 2    50   ~ 0
+Text Label 8150 4250 2    50   ~ 0
 GPIO26
 Wire Wire Line
 	4850 4800 5000 4800
-Text Label 8150 4250 2    50   ~ 0
-GPIO20(SPI1_MOSI)
 Wire Wire Line
 	8150 5550 8300 5550
@@
 	0    -1   -1   0
 $EndComp
-$Comp
-L power:GNDA #PWR0119
-U 1 1 5D245700
-P 9950 3600
-F 0 "#PWR0119" H 9950 3350 50  0001 C CNN
-F 1 "GNDA" H 9955 3427 50  0000 C CNN
-F 2 "" H 9950 3600 50  0001 C CNN
-F 3 "" H 9950 3600 50  0001 C CNN
-	1    9950 3600
-	1    0    0    -1
-$EndComp
-$Comp
-L power:GNDA #PWR0120
-U 1 1 5D25123E
-P 9950 4850
-F 0 "#PWR0120" H 9950 4600 50  0001 C CNN
-F 1 "GNDA" H 9955 4677 50  0000 C CNN
-F 2 "" H 9950 4850 50  0001 C CNN
-F 3 "" H 9950 4850 50  0001 C CNN
-	1    9950 4850
-	1    0    0    -1
-$EndComp
-$Comp
-L power:GNDA #PWR0121
-U 1 1 5D25C237
-P 9950 6150
-F 0 "#PWR0121" H 9950 5900 50  0001 C CNN
-F 1 "GNDA" H 9955 5977 50  0000 C CNN
-F 2 "" H 9950 6150 50  0001 C CNN
-F 3 "" H 9950 6150 50  0001 C CNN
-	1    9950 6150
-	1    0    0    -1
-$EndComp
-$Comp
-L power:GNDA #PWR0122
-U 1 1 5D2671CF
-P 6650 5400
-F 0 "#PWR0122" H 6650 5150 50  0001 C CNN
-F 1 "GNDA" H 6655 5227 50  0000 C CNN
-F 2 "" H 6650 5400 50  0001 C CNN
-F 3 "" H 6650 5400 50  0001 C CNN
-	1    6650 5400
-	1    0    0    -1
-$EndComp
-$Comp
-L power:GNDA #PWR0123
-U 1 1 5D2767E4
-P 6650 6650
-F 0 "#PWR0123" H 6650 6400 50  0001 C CNN
-F 1 "GNDA" H 6655 6477 50  0000 C CNN
-F 2 "" H 6650 6650 50  0001 C CNN
-F 3 "" H 6650 6650 50  0001 C CNN
-	1    6650 6650
-	1    0    0    -1
-$EndComp
-$Comp
-L power:GNDA #PWR0124
-U 1 1 5D282F37
-P 6650 4150
-F 0 "#PWR0124" H 6650 3900 50  0001 C CNN
-F 1 "GNDA" H 6655 3977 50  0000 C CNN
-F 2 "" H 6650 4150 50  0001 C CNN
-F 3 "" H 6650 4150 50  0001 C CNN
-	1    6650 4150
-	1    0    0    -1
-$EndComp
-$Comp
-L power:GNDA #PWR0125
-U 1 1 5D29294B
-P 6650 2850
-F 0 "#PWR0125" H 6650 2600 50  0001 C CNN
-F 1 "GNDA" H 6655 2677 50  0000 C CNN
-F 2 "" H 6650 2850 50  0001 C CNN
-F 3 "" H 6650 2850 50  0001 C CNN
-	1    6650 2850
-	1    0    0    -1
-$EndComp
-$Comp
-L power:GNDA #PWR0126
-U 1 1 5D29E75B
-P 6650 1600
-F 0 "#PWR0126" H 6650 1350 50  0001 C CNN
-F 1 "GNDA" H 6655 1427 50  0000 C CNN
-F 2 "" H 6650 1600 50  0001 C CNN
-F 3 "" H 6650 1600 50  0001 C CNN
-	1    6650 1600
-	1    0    0    -1
-$EndComp
-Text Label 4850 1000 2    50   ~ 0
-GPIO18(GEN1)(PWM0)
 Text Label 4850 2250 2    50   ~ 0
-GPIO17(GEN0)
-Text Label 4850 3550 2    50   ~ 0
 GPIO12(PWM0)
 Wire Wire Line
@@
 Wire Wire Line
 	9950 3500 9950 3600
-Text Label 4850 6050 2    50   ~ 0
-GPIO16
 Wire Wire Line
 	4850 6050 5000 6050
-Wire Wire Line
-	2400 1500 3450 1500
-Text Label 3450 1500 2    50   ~ 0
-GPIO18(GEN1)(PWM0)
 Text Label 750  1300 0    50   ~ 0
 ONE-WIRE
@@
 Text Label 750  2800 0    50   ~ 0
 GPIO26
-Text Label 750  2700 0    50   ~ 0
-GPIO19(SPI1_MISO)
-Text Label 750  2600 0    50   ~ 0
-GPIO13(PWM1)
-Text Label 750  2500 0    50   ~ 0
-GPIO6
-Text Label 750  2400 0    50   ~ 0
-GPIO5
-Text Label 750  1500 0    50   ~ 0
-GPIO17(GEN0)
 Text Label 750  1200 0    50   ~ 0
 GPIO3(SCL1)
@@
 Wire Wire Line
 	2400 2700 3450 2700
-Wire Wire Line
-	750  2800 1900 2800
-Wire Wire Line
-	750  2700 1900 2700
-Wire Wire Line
-	1900 2600 750  2600
-Wire Wire Line
-	750  2500 1900 2500
-Wire Wire Line
-	750  2400 1900 2400
-Wire Wire Line
-	1900 1500 750  1500
 Wire Wire Line
 	750  1300 1900 1300
@@
 	0    1    1    0
 $EndComp
-$Comp
-L power:GNDA #PWR0136
-U 1 1 5D93ABA2
-P 8300 2150
-F 0 "#PWR0136" H 8300 1900 50  0001 C CNN
-F 1 "GNDA" V 8305 2023 50  0000 R CNN
-F 2 "" H 8300 2150 50  0001 C CNN
-F 3 "" H 8300 2150 50  0001 C CNN
-	1    8300 2150
-	0    1    1    0
-$EndComp
 Wire Wire Line
 	8300 1750 9200 1750
@@
 	0    1    1    0
 $EndComp
+$Comp
+L power:GND #PWR0119
+U 1 1 5D924396
+P 8300 2150
+F 0 "#PWR0119" H 8300 1900 50  0001 C CNN
+F 1 "GND" V 8305 2022 50  0000 R CNN
+F 2 "" H 8300 2150 50  0001 C CNN
+F 3 "" H 8300 2150 50  0001 C CNN
+	1    8300 2150
+	0    1    1    0
+$EndComp
+$Comp
+L power:GND #PWR0120
+U 1 1 5D94A23B
+P 9950 3600
+F 0 "#PWR0120" H 9950 3350 50  0001 C CNN
+F 1 "GND" H 9955 3427 50  0000 C CNN
+F 2 "" H 9950 3600 50  0001 C CNN
+F 3 "" H 9950 3600 50  0001 C CNN
+	1    9950 3600
+	1    0    0    -1
+$EndComp
+$Comp
+L power:GND #PWR0121
+U 1 1 5D94C365
+P 9950 4850
+F 0 "#PWR0121" H 9950 4600 50  0001 C CNN
+F 1 "GND" H 9955 4677 50  0000 C CNN
+F 2 "" H 9950 4850 50  0001 C CNN
+F 3 "" H 9950 4850 50  0001 C CNN
+	1    9950 4850
+	1    0    0    -1
+$EndComp
+$Comp
+L power:GND #PWR0122
+U 1 1 5D95F49F
+P 9950 6150
+F 0 "#PWR0122" H 9950 5900 50  0001 C CNN
+F 1 "GND" H 9955 5977 50  0000 C CNN
+F 2 "" H 9950 6150 50  0001 C CNN
+F 3 "" H 9950 6150 50  0001 C CNN
+	1    9950 6150
+	1    0    0    -1
+$EndComp
+$Comp
+L power:GND #PWR0123
+U 1 1 5D96B5A0
+P 6650 6650
+F 0 "#PWR0123" H 6650 6400 50  0001 C CNN
+F 1 "GND" H 6655 6477 50  0000 C CNN
+F 2 "" H 6650 6650 50  0001 C CNN
+F 3 "" H 6650 6650 50  0001 C CNN
+	1    6650 6650
+	1    0    0    -1
+$EndComp
+$Comp
+L power:GND #PWR0124
+U 1 1 5D9798D2
+P 6650 5400
+F 0 "#PWR0124" H 6650 5150 50  0001 C CNN
+F 1 "GND" H 6655 5227 50  0000 C CNN
+F 2 "" H 6650 5400 50  0001 C CNN
+F 3 "" H 6650 5400 50  0001 C CNN
+	1    6650 5400
+	1    0    0    -1
+$EndComp
+$Comp
+L power:GND #PWR0125
+U 1 1 5D98C248
+P 6650 4150
+F 0 "#PWR0125" H 6650 3900 50  0001 C CNN
+F 1 "GND" H 6655 3977 50  0000 C CNN
+F 2 "" H 6650 4150 50  0001 C CNN
+F 3 "" H 6650 4150 50  0001 C CNN
+	1    6650 4150
+	1    0    0    -1
+$EndComp
+$Comp
+L power:GND #PWR0126
+U 1 1 5D99A370
+P 6650 2850
+F 0 "#PWR0126" H 6650 2600 50  0001 C CNN
+F 1 "GND" H 6655 2677 50  0000 C CNN
+F 2 "" H 6650 2850 50  0001 C CNN
+F 3 "" H 6650 2850 50  0001 C CNN
+	1    6650 2850
+	1    0    0    -1
+$EndComp
+$Comp
+L power:GND #PWR0136
+U 1 1 5D9B74EF
+P 6650 1600
+F 0 "#PWR0136" H 6650 1350 50  0001 C CNN
+F 1 "GND" H 6655 1427 50  0000 C CNN
+F 2 "" H 6650 1600 50  0001 C CNN
+F 3 "" H 6650 1600 50  0001 C CNN
+	1    6650 1600
+	1    0    0    -1
+$EndComp
+NoConn ~ 1900 1500
+NoConn ~ 2400 1500
+Wire Wire Line
+	750  2400 1900 2400
+Wire Wire Line
+	750  2500 1900 2500
+Wire Wire Line
+	1900 2600 750  2600
+Wire Wire Line
+	750  2700 1900 2700
+Wire Wire Line
+	750  2800 1900 2800
+Text Label 750  2400 0    50   ~ 0
+GPIO5
+Text Label 750  2500 0    50   ~ 0
+GPIO6
+Text Label 750  2600 0    50   ~ 0
+GPIO13(PWM1)
+Text Label 750  2700 0    50   ~ 0
+GPIO19(SPI1_MISO)
+Text Label 4850 1000 2    50   ~ 0
+GPIO6
+Text Label 4850 4800 2    50   ~ 0
+GPIO16
+Text Label 8150 5550 2    50   ~ 0
+GPIO21(SPI1_SCK)
+Text Label 8150 3000 2    50   ~ 0
+GPIO20(SPI1_MOSI)
 $EndSCHEMATC

Commit message: final version
Parts:
- added J1: Conn_01x09, Connector_PinSocket_2.54mm:PinSocket_1x09_P2.54mm_Vertical, symbol Connector_Generic:Conn_01x09
- added SW1: SW_Push, Button_Switch_SMD:SW_Push_SPST_NO_Alps_SKRK, symbol Switch:SW_Push
- D1, D2, D3, D4, D5, D6, D7, D8: footprint Diode_THT:D_DO-41_SOD81_P3.81mm_Vertical_KathodeUp -> Diode_THT:D_DO-41_SOD81_P3.81mm_Vertical_AnodeUp
- renumbered J1 to J2, J2 to J4, R11 to R10, R12 to R11, R10 to R12, R9 to R13, R13 to R3, R3 to R4, R4 to R5, R5 to R6, R6 to R7, R7 to R8, R8 to R9
Connections:
- net GNDA is gone; now on net GND: J4.3 (Pin_3)
- net +3V3: now also J1.8 (Pin_8); no longer P1.17 (Pin_17)
- net GND: now also D1.2 (A), D2.2 (A), D3.2 (A), D4.2 (A), D5.2 (A), D6.2 (A), D7.2 (A), D8.2 (A), J1.7 (Pin_7), SW1.2; no longer D1.1 (K), D2.1 (K), D3.1 (K), D4.1 (K), D5.1 (K), D6.1 (K), D7.1 (K), D8.1 (K)
- net GPIO14(TXD0): now also J1.6 (Pin_6)
- net GPIO15(RXD0): now also J1.5 (Pin_5)
- net NOISE-DIODE: now also D8.1 (K); no longer D8.2 (A)
- net POS1: now also D1.1 (K); no longer D1.2 (A)
- net POS2: now also D2.1 (K); no longer D2.2 (A)
- net POS3: now also D3.1 (K); no longer D3.2 (A)
- net POS4: now also D4.1 (K); no longer D4.2 (A)
- net POS5: now also D5.1 (K); no longer D5.2 (A)
- net POS6: now also D6.1 (K); no longer D6.2 (A)
- net RESET: now also D7.1 (K); no longer D7.2 (A)
- net at U9.4 (~RST): now also SW1.1
- net +5V: no longer names the net of P1.2 (Pin_2)
- net +5V: no longer P1.4 (Pin_4)
- no-connect marks 14 -> 22
Other:
- moved on the sheet: BT1, C1, J3, J4, R10, R11, R12, R13, U9
