File: switch-control-hat/prizm-switch-control.kicad_pcb (KiCad board)
At the start: 2 copper layers, 85 x 56 mm, 45 parts, among them J1 Power Connector, J2 Frontend Connector, P1 RPi-Header, U1 MCP23017_SO, U10 TLP3543, U11 TLP3543, U12 TLP3543, U2 DS3231M, U3 TLP3543, U4 TLP3543, U5 TLP3543, U6 TLP3543, U7 TLP3543, U8 TLP3543, U9 TLP3543

Commit message: Fixed ERC and DRC errors
Parts:
- BT1: value 3V -> V3
Connections:
- net Net-(BT1-Pad1) renamed /real_time_clock/3.3V_Backup
