File: switch-control-hat/rpi.sch (KiCad schematic (older format))
At the start: 8 parts, among them J1 Power Connector, P1 RPi-Header

Commit message: Fixed ERC and DRC errors
Parts:
- MK1, MK2, MK3, MK4: symbol switch-control-hat-rescue:Mounting_Hole-Mechanical -> Mechanical:MountingHole
Other:
- moved on the sheet: J1, MK1, MK2, MK3, MK4, P1, R1, R2
